File: LinkPlug.kicad_sch (KiCad schematic)
At the start: 4 parts, among them J901 NE8FAH, U901 THVD24x2

Commit message: Update
Other:
- note added: "PoE Passive +24V IEEE 802.3af Mode B"
- note added: "RS-422 3MHz"
Changed lines of the file:
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@@
 		(company "Plug")
+	)
+	(text "RS-422 3MHz"
+		(exclude_from_sim no)
+		(at 170.942 107.696 0)
+		(effects
+			(font
+				(size 1.27 1.27)
+			)
+		)
+	)
+	(text "PoE Passive +24V\nIEEE 802.3af Mode B"
+		(exclude_from_sim no)
+		(at 163.83 158.496 0)
+		(effects
+			(font
+				(size 1.27 1.27)
+			)
+			(justify left)
+		)
 	)
 	(junction
@@
 		(mirror y)
 		(unit 1)
-		(exclude_from_sim no)
+		(exclude_from_sim yes)
 		(in_bom yes)
 		(on_board yes)
@@
 			(at 148.59 134.62 0)
 			(effects
-				(font
-					(size 1.27 1.27)
-				)
-				(hide yes)
-			)
-		)
-		(property "Sim.Enable" "0"
-			(at 148.59 134.62 0)
-			(effects

Commit message: Update parts
Parts:
- C901: footprint Capacitor_SMD:C_0603_1608Metric -> V2_Capacitor_SMD:C_0603; symbol Device:C_Small -> V2_Device:C_0603_0u1; Manufacturer (none) -> TDK; Mouser (none) -> 810-CGA3E2X7R1H104MA; Product (none) -> CGA3E2X7R1H104M080AA
- J901: value NE8FAH -> NE8FAV; Manfacturer (none) -> Neutrik; Manufacturer (none) -> Neutrik; Mouser (none) -> 568-NE8FAV-SD; Product (none) -> NE8FAV-SD
- R901: footprint Resistor_SMD:R_0603_1608Metric -> V2_Resistor_SMD:R_0603; symbol Device:R_Small -> V2_Device:R_0603_100R; Manufacturer (none) -> Vishay; Mouser (none) -> 71-CRCW0603100RFKEAH; Product (none) -> CRCW0603100RFKEAHP; Rating (none) -> 330mW
- U901: value THVD24x2 -> THVD2442; symbol V2_Interface_RS485:THVD24x2 -> V2_Interface_RS485:THVD2442; Manufacturer (none) -> Texas Instruments; Mouser (none) -> 595-THVD2442DRCR; Product (none) -> THVD2442DRCR
Changed lines of the file:
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@@
 	)
 	(symbol
-		(lib_id "power:GND")
+		(lib_id "V2_power:GND")
 		(at 168.91 71.12 0)
 		(unit 1)
@@
 	)
 	(symbol
-		(lib_id "V2_Interface_RS485:THVD24x2")
+		(lib_id "V2_Interface_RS485:THVD2442")
 		(at 148.59 88.9 0)
 		(unit 1)
@@
 			)
 		)
-		(property "Value" "THVD24x2"
+		(property "Value" "THVD2442"
 			(at 150.7333 73.66 0)
 			(effects
@@
 		(property "Description" ""
 			(at 148.59 88.9 0)
+			(effects
+				(font
+					(size 1.27 1.27)
+				)
+				(hide yes)
+			)
+		)
+		(property "Mouser" "595-THVD2442DRCR"
+			(at 148.59 88.9 0)
+			(effects
+				(font
+					(size 1.27 1.27)
+				)
+				(hide yes)
+			)
+		)
+		(property "Sim.Pin" ""
+			(at 148.59 88.9 0)
+			(effects
+				(font
+					(size 1.27 1.27)
+				)
+				(hide yes)
+			)
+		)
+		(property "Product" "THVD2442DRCR "
+			(at 148.59 121.92 0)
+			(effects
+				(font
+					(size 1.27 1.27)
+				)
+				(hide yes)
+			)
+		)
+		(property "Manufacturer" "Texas Instruments"
+			(at 148.59 119.38 0)
 			(effects
 				(font
@@
 	)
 	(symbol
-		(lib_id "Device:R_Small")
+		(lib_id "V2_Device:R_0603_100R")
 		(at 161.29 83.82 0)
 		(unit 1)
@@
 		)
 		(property "Value" "100R"
-			(at 166.37 85.09 0)
-			(effects
-				(font
-					(size 1.27 1.27)
-				)
-			)
-		)
-		(property "Footprint" "Resistor_SMD:R_0603_1608Metric"
+			(at 165.1 85.09 0)
+			(effects
+				(font
+					(size 1.27 1.27)
+				)
+			)
+		)
+		(property "Footprint" "V2_Resistor_SMD:R_0603"
+			(at 161.29 99.568 0)
+			(effects
+				(font
+					(size 1.27 1.27)
+				)
+				(hide yes)
+			)
+		)
+		(property "Datasheet" ""
 			(at 161.29 83.82 0)
 			(effects
@@
 			)
 		)
-		(property "Datasheet" "~"
+		(property "Description" "Resistor, small symbol"
+			(at 161.29 96.012 0)
+			(effects
+				(font
+					(size 1.27 1.27)
+				)
+				(hide yes)
+			)
+		)
+		(property "Mouser" "71-CRCW0603100RFKEAH"
+			(at 161.29 99.314 0)
+			(effects
+				(font
+					(size 1.27 1.27)
+				)
+				(hide yes)
+			)
+		)
+		(property "Sim.Pin" ""
 			(at 161.29 83.82 0)
 			(effects
@@
 			)
 		)
-		(property "Description" "Resistor, small symbol"
-			(at 161.29 83.82 0)
+		(property "Rating" "330mW"
+			(at 161.29 106.68 0)
+			(effects
+				(font
+					(size 1.27 1.27)
+				)
+				(hide yes)
+			)
+		)
+		(property "Manufacturer" "Vishay"
+			(at 161.29 101.6 0)
+			(effects
+				(font
+					(size 1.27 1.27)
+				)
+				(hide yes)
+			)
+		)
+		(property "Product" "CRCW0603100RFKEAHP"
+			(at 161.29 104.14 0)
 			(effects
 				(font
@@
 		(mirror y)
 		(unit 1)
-		(exclude_from_sim yes)
+		(exclude_from_sim no)
 		(in_bom yes)
 		(on_board yes)
@@
 			)
 		)
-		(property "Value" "NE8FAH"
+		(property "Value" "NE8FAV"
 			(at 148.59 119.38 0)
 			(effects
@@
 		(property "Description" ""
 			(at 148.59 134.62 0)
+			(effects
+				(font
+					(size 1.27 1.27)
+				)
+				(hide yes)
+			)
+		)
+		(property "Mouser" "568-NE8FAV-SD"
+			(at 148.59 159.512 0)
+			(effects
+				(font
+					(size 1.27 1.27)
+				)
+				(hide yes)
+			)
+		)
+		(property "Sim.Pin" ""
+			(at 148.59 134.62 0)
+			(effects
+				(font
+					(size 1.27 1.27)
+				)
+				(hide yes)
+			)
+		)
+		(property "Manfacturer" "Neutrik"
+			(at 148.59 160.02 0)
+			(effects
+				(font
+					(size 1.27 1.27)
+				)
+				(hide yes)
+			)
+		)
+		(property "Product" "NE8FAV-SD"
+			(at 148.59 162.56 0)
+			(effects
+				(font
+					(size 1.27 1.27)
+				)
+				(hide yes)
+			)
+		)
+		(property "Manufacturer" "Neutrik"
+			(at 148.59 160.02 0)
 			(effects
 				(font
@@
 	)
 	(symbol
-		(lib_id "power:GND")
+		(lib_id "V2_power:GND")
 		(at 149.86 104.14 0)
 		(unit 1)
@@
 	)
 	(symbol
-		(lib_id "power:+3V3")
+		(lib_id "V2_power:+3V3")
 		(at 148.59 66.04 0)
 		(unit 1)
@@
 	)
 	(symbol
-		(lib_id "Device:C_Small")
+		(lib_id "V2_Device:C_0603_0u1")
 		(at 168.91 68.58 0)
 		(unit 1)
@@
 			)
 		)
-		(property "Footprint" "Capacitor_SMD:C_0603_1608Metric"
+		(property "Footprint" "V2_Capacitor_SMD:C_0603"
+			(at 168.91 85.598 0)
+			(effects
+				(font
+					(size 1.27 1.27)
+				)
+				(hide yes)
+			)
+		)
+		(property "Datasheet" ""
 			(at 168.91 68.58 0)
 			(effects
@@
 			)
 		)
-		(property "Datasheet" "~"
+		(property "Description" "Unpolarized capacitor, small symbol"
+			(at 168.91 82.042 0)
+			(effects
+				(font
+					(size 1.27 1.27)
+				)
+				(hide yes)
+			)
+		)
+		(property "Mouser" "810-CGA3E2X7R1H104MA"
+			(at 168.91 85.852 0)
+			(effects
+				(font
+					(size 1.27 1.27)
+				)
+				(hide yes)
+			)
+		)
+		(property "Sim.Pin" ""
 			(at 168.91 68.58 0)
 			(effects
@@
 			)
 		)
-		(property "Description" "Unpolarized capacitor, small symbol"
-			(at 168.91 68.58 0)
+		(property "Manufacturer" "TDK"
+			(at 168.91 83.82 0)
+			(effects
+				(font
+					(size 1.27 1.27)
+				)
+				(hide yes)
+			)
+		)
+		(property "Product" "CGA3E2X7R1H104M080AA"
+			(at 168.91 86.36 0)
 			(effects
 				(font
@@
 	)
 	(symbol
-		(lib_id "power:GND")
+		(lib_id "V2_power:GND")
 		(at 138.43 124.46 270)
 		(mirror x)

Commit message: Update library
Parts:
- C901: Rating (none) -> 50V
- J901: Manfacturer Neutrik -> (none)
Changed lines of the file:
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@@
 			)
 		)
-		(property "Description" "Power symbol creates a global label with name \"GND\" , ground"
+		(property "Description" ""
 			(at 168.91 71.12 0)
 			(effects
@@
 			)
 		)
-		(property "Sim.Pin" ""
-			(at 148.59 88.9 0)
-			(effects
-				(font
-					(size 1.27 1.27)
-				)
-				(hide yes)
-			)
-		)
 		(property "Product" "THVD2442DRCR "
 			(at 148.59 121.92 0)
@@
 		(property "Mouser" "71-CRCW0603100RFKEAH"
 			(at 161.29 99.314 0)
-			(effects
-				(font
-					(size 1.27 1.27)
-				)
-				(hide yes)
-			)
-		)
-		(property "Sim.Pin" ""
-			(at 161.29 83.82 0)
 			(effects
 				(font
@@
 			)
 		)
-		(property "Sim.Pin" ""
-			(at 148.59 134.62 0)
-			(effects
-				(font
-					(size 1.27 1.27)
-				)
-				(hide yes)
-			)
-		)
-		(property "Manfacturer" "Neutrik"
-			(at 148.59 160.02 0)
-			(effects
-				(font
-					(size 1.27 1.27)
-				)
-				(hide yes)
-			)
-		)
 		(property "Product" "NE8FAV-SD"
 			(at 148.59 162.56 0)
@@
 			)
 		)
-		(property "Description" "Power symbol creates a global label with name \"GND\" , ground"
+		(property "Description" ""
 			(at 149.86 104.14 0)
 			(effects
@@
 			)
 		)
-		(property "Description" "Power symbol creates a global label with name \"+3V3\""
+		(property "Description" ""
 			(at 148.59 66.04 0)
 			(effects
@@
 			)
 		)
-		(property "Sim.Pin" ""
-			(at 168.91 68.58 0)
-			(effects
-				(font
-					(size 1.27 1.27)
-				)
-				(hide yes)
-			)
-		)
 		(property "Manufacturer" "TDK"
 			(at 168.91 83.82 0)
@@
 		(property "Product" "CGA3E2X7R1H104M080AA"
 			(at 168.91 86.36 0)
+			(effects
+				(font
+					(size 1.27 1.27)
+				)
+				(hide yes)
+			)
+		)
+		(property "Rating" "50V"
+			(at 168.91 91.44 0)
 			(effects
 				(font
@@
 			)
 		)
-		(property "Description" "Power symbol creates a global label with name \"GND\" , ground"
+		(property "Description" ""
 			(at 138.43 124.46 0)
 			(effects

Commit message: Update Library
Parts:
- C901: symbol V2_Device:C_0603_0u1 -> V2_Capacitor:0603_0u1
- R901: symbol V2_Device:R_0603_100R -> V2_Resistor:0603_100R
Changed lines of the file:
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@@
 	)
 	(symbol
-		(lib_id "V2_Device:R_0603_100R")
+		(lib_id "V2_Resistor:0603_100R")
 		(at 161.29 83.82 0)
 		(unit 1)
@@
 	)
 	(symbol
-		(lib_id "V2_Device:C_0603_0u1")
+		(lib_id "V2_Capacitor:0603_0u1")
 		(at 168.91 68.58 0)
 		(unit 1)

Commit message: Refresh
Other:
- note added: "PoE Passive +28V IEEE 802.3af Mode B"
- note removed: "PoE Passive +24V IEEE 802.3af Mode B"
Changed lines of the file:
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@@
 		)
 	)
-	(text "PoE Passive +24V\nIEEE 802.3af Mode B"
+	(text "PoE Passive +28V\nIEEE 802.3af Mode B"
 		(exclude_from_sim no)
 		(at 163.83 158.496 0)
@@
 		(dnp no)
 		(property "Reference" "R901"
-			(at 166.37 82.55 0)
+			(at 165.862 82.55 0)
 			(effects
 				(font
@@
 		)
 		(property "Value" "100R"
-			(at 165.1 85.09 0)
-			(effects
-				(font
+			(at 165.862 84.836 0)
+			(effects
+				(font

Commit message: Replace diode
Other:
- title: V2 Link -> V2 drum

Commit message: Update
Parts:
- C901: Id (none) -> Capacitor:${SYMBOL_NAME}
- J901: Id (none) -> EtherCon:${SYMBOL_NAME}; Rating (none) -> CAT5e
- R901: Id (none) -> Resistor:${SYMBOL_NAME}
- U901: Id (none) -> RS485:${SYMBOL_NAME}; Rating (none) -> 20Mbps
Other:
- company: Plug -> Versio Duo
Changed lines of the file:
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@@
 	(title_block
 		(title "V2 drum")
-		(date "2026-03-30")
+		(date "2026-04-14")
 		(rev "2026-03-30")
-		(company "Plug")
+		(company "Versio Duo")
+		(comment 1 "Percussion Controller")
 	)
 	(text "RS-422 3MHz"
@@
 		(in_pos_files yes)
 		(dnp no)
-		(property "Reference" "#PWR902"
+		(property "Reference" "#PWR0904"
 			(at 168.91 77.47 0)
 			(hide yes)
@@
 			(project "drum"
 				(path "/6c8448b4-b04d-47e1-934e-e40cbe27a7be/c6db2f80-f80f-4104-8ca1-02f0ab85cfea"
-					(reference "#PWR902")
+					(reference "#PWR0904")
 					(unit 1)
 				)
@@
 			)
 		)
+		(property "Id" "RS485:${SYMBOL_NAME}"
+			(at 148.59 120.65 0)
+			(hide yes)
+			(show_name no)
+			(do_not_autoplace no)
+			(effects
+				(font
+					(size 1.27 1.27)
+				)
+			)
+		)
+		(property "Rating" "20Mbps"
+			(at 149.86 128.27 0)
+			(hide yes)
+			(show_name no)
+			(do_not_autoplace no)
+			(effects
+				(font
+					(size 1.27 1.27)
+				)
+			)
+		)
 		(pin "1"
 		)
@@
 		(property "Product" "CRCW0603100RFKEAHP"
 			(at 161.29 104.14 0)
+			(hide yes)
+			(show_name no)
+			(do_not_autoplace no)
+			(effects
+				(font
+					(size 1.27 1.27)
+				)
+			)
+		)
+		(property "Id" "Resistor:${SYMBOL_NAME}"
+			(at 161.29 97.79 0)
 			(hide yes)
 			(show_name no)
@@
 			)
 		)
+		(property "Id" "EtherCon:${SYMBOL_NAME}"
+			(at 148.59 167.64 0)
+			(hide yes)
+			(show_name no)
+			(do_not_autoplace no)
+			(effects
+				(font
+					(size 1.27 1.27)
+				)
+			)
+		)
+		(property "Rating" "CAT5e"
+			(at 148.59 170.18 0)
+			(hide yes)
+			(show_name no)
+			(do_not_autoplace no)
+			(effects
+				(font
+					(size 1.27 1.27)
+				)
+			)
+		)
 		(pin "7"
 		)
@@
 		(in_pos_files yes)
 		(dnp no)
-		(property "Reference" "#PWR903"
+		(property "Reference" "#PWR0903"
 			(at 149.86 110.49 0)
 			(hide yes)
@@
 			(project "drum"
 				(path "/6c8448b4-b04d-47e1-934e-e40cbe27a7be/c6db2f80-f80f-4104-8ca1-02f0ab85cfea"
-					(reference "#PWR903")
+					(reference "#PWR0903")
 					(unit 1)
 				)
@@
 		(in_pos_files yes)
 		(dnp no)
-		(property "Reference" "#PWR901"
+		(property "Reference" "#PWR0902"
 			(at 148.59 69.85 0)
 			(hide yes)
@@
 			(project "drum"
 				(path "/6c8448b4-b04d-47e1-934e-e40cbe27a7be/c6db2f80-f80f-4104-8ca1-02f0ab85cfea"
-					(reference "#PWR901")
+					(reference "#PWR0902")
 					(unit 1)
 				)
@@
 			)
 		)
+		(property "Id" "Capacitor:${SYMBOL_NAME}"
+			(at 168.91 83.82 0)
+			(hide yes)
+			(show_name no)
+			(do_not_autoplace no)
+			(effects
+				(font
+					(size 1.27 1.27)
+				)
+			)
+		)
 		(pin "1"
 		)
@@
 		(in_pos_files yes)
 		(dnp no)
-		(property "Reference" "#PWR904"
+		(property "Reference" "#PWR0901"
 			(at 132.08 124.46 0)
 			(hide yes)
@@
 			(project "drum"
 				(path "/6c8448b4-b04d-47e1-934e-e40cbe27a7be/c6db2f80-f80f-4104-8ca1-02f0ab85cfea"
-					(reference "#PWR904")
+					(reference "#PWR0901")
 					(unit 1)
 				)
