File: LinkPlug.kicad_sch (KiCad schematic)
At the start: 4 parts, among them J901 NE8FAV, U901 THVD2442

Commit message: Good Bye Imperial
Parts:
- C901: footprint V2_Capacitor_SMD:C_0603 -> V2_Capacitor_SMD:C_1608; symbol V2_Capacitor:0603_0u1 -> V2_Capacitor:1608_0u1
- R901: footprint V2_Resistor_SMD:R_0603 -> V2_Resistor_SMD:R_1608; symbol V2_Resistor:0603_100R -> V2_Resistor:1608_100R
Changed lines of the file:
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@@
 	(title_block
 		(title "V2 drum")
-		(date "2026-04-14")
+		(date "2026-05-11")
 		(rev "2026-03-30")
 		(company "Versio Duo")
@@
 	)
 	(symbol
-		(lib_id "V2_Resistor:0603_100R")
+		(lib_id "V2_Resistor:1608_100R")
 		(at 161.29 83.82 0)
 		(unit 1)
@@
 			)
 		)
-		(property "Footprint" "V2_Resistor_SMD:R_0603"
+		(property "Footprint" "V2_Resistor_SMD:R_1608"
 			(at 161.29 99.568 0)
 			(hide yes)
@@
 	)
 	(symbol
-		(lib_id "V2_Capacitor:0603_0u1")
+		(lib_id "V2_Capacitor:1608_0u1")
 		(at 168.91 68.58 0)
 		(unit 1)
@@
 			)
 		)
-		(property "Footprint" "V2_Capacitor_SMD:C_0603"
+		(property "Footprint" "V2_Capacitor_SMD:C_1608"
 			(at 168.91 85.598 0)
 			(hide yes)
