File: LinkSocket.kicad_sch (KiCad schematic)
At the start: 4 parts, among them J1001 NE8FAH, U1001 THVD24x2

Commit message: Update
Other:
- note added: "PoE Passive +24V IEEE 802.3af Mode B"
- note added: "RS-422 3MHz"
Changed lines of the file:
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@@
 		(company "Socket")
+	)
+	(text "PoE Passive +24V\nIEEE 802.3af Mode B"
+		(exclude_from_sim no)
+		(at 169.164 150.876 0)
+		(effects
+			(font
+				(size 1.27 1.27)
+			)
+			(justify left)
+		)
+	)
+	(text "RS-422 3MHz"
+		(exclude_from_sim no)
+		(at 176.022 98.298 0)
+		(effects
+			(font
+				(size 1.27 1.27)
+			)
+		)
 	)
 	(junction
@@
 		(mirror y)
 		(unit 1)
-		(exclude_from_sim no)
+		(exclude_from_sim yes)
 		(in_bom yes)
 		(on_board yes)
@@
 			(at 154.94 128.27 0)
 			(effects
-				(font
-					(size 1.27 1.27)
-				)
-				(hide yes)
-			)
-		)
-		(property "Sim.Enable" "0"
-			(at 154.94 128.27 0)
-			(effects

Commit message: Update parts
Parts:
- C1001: footprint Capacitor_SMD:C_0603_1608Metric -> V2_Capacitor_SMD:C_0603; symbol Device:C_Small -> V2_Device:C_0603_0u1; Manufacturer (none) -> TDK; Mouser (none) -> 810-CGA3E2X7R1H104MA; Product (none) -> CGA3E2X7R1H104M080AA
- J1001: value NE8FAH -> NE8FAV; Manfacturer (none) -> Neutrik; Manufacturer (none) -> Neutrik; Mouser (none) -> 568-NE8FAV-SD; Product (none) -> NE8FAV-SD
- R1001: footprint Resistor_SMD:R_0603_1608Metric -> V2_Resistor_SMD:R_0603; symbol Device:R_Small -> V2_Device:R_0603_100R; Manufacturer (none) -> Vishay; Mouser (none) -> 71-CRCW0603100RFKEAH; Product (none) -> CRCW0603100RFKEAHP; Rating (none) -> 330mW
- U1001: value THVD24x2 -> THVD2442; symbol V2_Interface_RS485:THVD24x2 -> V2_Interface_RS485:THVD2442; Manufacturer (none) -> Texas Instruments; Mouser (none) -> 595-THVD2442DRCR; Product (none) -> THVD2442DRCR
Changed lines of the file:
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@@
 	)
 	(symbol
-		(lib_id "power:+3V3")
+		(lib_id "V2_power:+3V3")
 		(at 154.94 58.42 0)
 		(unit 1)
@@
 	)
 	(symbol
-		(lib_id "V2_Interface_RS485:THVD24x2")
+		(lib_id "V2_Interface_RS485:THVD2442")
 		(at 154.94 81.28 0)
 		(unit 1)
@@
 			)
 		)
-		(property "Value" "THVD24x2"
+		(property "Value" "THVD2442"
 			(at 156.8959 66.04 0)
 			(effects
@@
 		(property "Description" ""
 			(at 154.94 81.28 0)
+			(effects
+				(font
+					(size 1.27 1.27)
+				)
+				(hide yes)
+			)
+		)
+		(property "Mouser" "595-THVD2442DRCR"
+			(at 154.94 81.28 0)
+			(effects
+				(font
+					(size 1.27 1.27)
+				)
+				(hide yes)
+			)
+		)
+		(property "Sim.Pin" ""
+			(at 154.94 81.28 0)
+			(effects
+				(font
+					(size 1.27 1.27)
+				)
+				(hide yes)
+			)
+		)
+		(property "Product" "THVD2442DRCR "
+			(at 154.94 114.3 0)
+			(effects
+				(font
+					(size 1.27 1.27)
+				)
+				(hide yes)
+			)
+		)
+		(property "Manufacturer" "Texas Instruments"
+			(at 154.94 111.76 0)
 			(effects
 				(font
@@
 		(mirror y)
 		(unit 1)
-		(exclude_from_sim yes)
+		(exclude_from_sim no)
 		(in_bom yes)
 		(on_board yes)
@@
 			)
 		)
-		(property "Value" "NE8FAH"
+		(property "Value" "NE8FAV"
 			(at 154.94 113.03 0)
 			(effects
@@
 		(property "Description" ""
 			(at 154.94 128.27 0)
+			(effects
+				(font
+					(size 1.27 1.27)
+				)
+				(hide yes)
+			)
+		)
+		(property "Mouser" "568-NE8FAV-SD"
+			(at 154.94 153.162 0)
+			(effects
+				(font
+					(size 1.27 1.27)
+				)
+				(hide yes)
+			)
+		)
+		(property "Sim.Pin" ""
+			(at 154.94 128.27 0)
+			(effects
+				(font
+					(size 1.27 1.27)
+				)
+				(hide yes)
+			)
+		)
+		(property "Manfacturer" "Neutrik"
+			(at 154.94 153.67 0)
+			(effects
+				(font
+					(size 1.27 1.27)
+				)
+				(hide yes)
+			)
+		)
+		(property "Product" "NE8FAV-SD"
+			(at 154.94 156.21 0)
+			(effects
+				(font
+					(size 1.27 1.27)
+				)
+				(hide yes)
+			)
+		)
+		(property "Manufacturer" "Neutrik"
+			(at 154.94 153.67 0)
 			(effects
 				(font
@@
 	)
 	(symbol
-		(lib_id "power:GND")
+		(lib_id "V2_power:GND")
 		(at 154.94 96.52 0)
 		(unit 1)
@@
 	)
 	(symbol
-		(lib_id "power:GND")
+		(lib_id "V2_power:GND")
 		(at 176.53 63.5 0)
 		(unit 1)
@@
 	)
 	(symbol
-		(lib_id "Device:R_Small")
+		(lib_id "V2_Device:R_0603_100R")
 		(at 167.64 76.2 0)
 		(unit 1)
@@
 		)
 		(property "Value" "100R"
-			(at 172.72 77.47 0)
-			(effects
-				(font
-					(size 1.27 1.27)
-				)
-			)
-		)
-		(property "Footprint" "Resistor_SMD:R_0603_1608Metric"
+			(at 171.45 77.47 0)
+			(effects
+				(font
+					(size 1.27 1.27)
+				)
+			)
+		)
+		(property "Footprint" "V2_Resistor_SMD:R_0603"
+			(at 167.64 91.948 0)
+			(effects
+				(font
+					(size 1.27 1.27)
+				)
+				(hide yes)
+			)
+		)
+		(property "Datasheet" ""
 			(at 167.64 76.2 0)
 			(effects
@@
 			)
 		)
-		(property "Datasheet" "~"
+		(property "Description" "Resistor, small symbol"
+			(at 167.64 88.392 0)
+			(effects
+				(font
+					(size 1.27 1.27)
+				)
+				(hide yes)
+			)
+		)
+		(property "Mouser" "71-CRCW0603100RFKEAH"
+			(at 167.64 91.694 0)
+			(effects
+				(font
+					(size 1.27 1.27)
+				)
+				(hide yes)
+			)
+		)
+		(property "Sim.Pin" ""
 			(at 167.64 76.2 0)
 			(effects
@@
 			)
 		)
-		(property "Description" "Resistor, small symbol"
-			(at 167.64 76.2 0)
+		(property "Rating" "330mW"
+			(at 167.64 99.06 0)
+			(effects
+				(font
+					(size 1.27 1.27)
+				)
+				(hide yes)
+			)
+		)
+		(property "Manufacturer" "Vishay"
+			(at 167.64 93.98 0)
+			(effects
+				(font
+					(size 1.27 1.27)
+				)
+				(hide yes)
+			)
+		)
+		(property "Product" "CRCW0603100RFKEAHP"
+			(at 167.64 96.52 0)
 			(effects
 				(font
@@
 	)
 	(symbol
-		(lib_id "power:GND")
+		(lib_id "V2_power:GND")
 		(at 143.51 118.11 270)
 		(mirror x)
@@
 	)
 	(symbol
-		(lib_id "Device:C_Small")
+		(lib_id "V2_Device:C_0603_0u1")
 		(at 176.53 60.96 0)
 		(unit 1)
@@
 			)
 		)
-		(property "Footprint" "Capacitor_SMD:C_0603_1608Metric"
+		(property "Footprint" "V2_Capacitor_SMD:C_0603"
+			(at 176.53 77.978 0)
+			(effects
+				(font
+					(size 1.27 1.27)
+				)
+				(hide yes)
+			)
+		)
+		(property "Datasheet" ""
 			(at 176.53 60.96 0)
 			(effects
@@
 			)
 		)
-		(property "Datasheet" "~"
+		(property "Description" "Unpolarized capacitor, small symbol"
+			(at 176.53 74.422 0)
+			(effects
+				(font
+					(size 1.27 1.27)
+				)
+				(hide yes)
+			)
+		)
+		(property "Mouser" "810-CGA3E2X7R1H104MA"
+			(at 176.53 78.232 0)
+			(effects
+				(font
+					(size 1.27 1.27)
+				)
+				(hide yes)
+			)
+		)
+		(property "Sim.Pin" ""
 			(at 176.53 60.96 0)
 			(effects
@@
 			)
 		)
-		(property "Description" "Unpolarized capacitor, small symbol"
-			(at 176.53 60.96 0)
-			(effects
-				(font
+		(property "Manufacturer" "TDK"
+			(at 176.53 76.2 0)
+			(effects
+				(font
+					(size 1.27 1.27)
+				)
+				(hide yes)
+			)
+		)
+		(property "Product" "CGA3E2X7R1H104M080AA"
+			(at 176.53 78.74 0)
+			(effects
+				(font

Commit message: Update library
Parts:
- C1001: Rating (none) -> 50V
- J1001: Manfacturer Neutrik -> (none)
Changed lines of the file:
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@@
 			)
 		)
-		(property "Description" "Power symbol creates a global label with name \"+3V3\""
+		(property "Description" ""
 			(at 154.94 58.42 0)
 			(effects
@@
 		)
 		(property "Mouser" "595-THVD2442DRCR"
-			(at 154.94 81.28 0)
-			(effects
-				(font
-					(size 1.27 1.27)
-				)
-				(hide yes)
-			)
-		)
-		(property "Sim.Pin" ""
 			(at 154.94 81.28 0)
 			(effects
@@
 			)
 		)
-		(property "Sim.Pin" ""
-			(at 154.94 128.27 0)
-			(effects
-				(font
-					(size 1.27 1.27)
-				)
-				(hide yes)
-			)
-		)
-		(property "Manfacturer" "Neutrik"
-			(at 154.94 153.67 0)
-			(effects
-				(font
-					(size 1.27 1.27)
-				)
-				(hide yes)
-			)
-		)
 		(property "Product" "NE8FAV-SD"
 			(at 154.94 156.21 0)
@@
 			)
 		)
-		(property "Description" "Power symbol creates a global label with name \"GND\" , ground"
+		(property "Description" ""
 			(at 154.94 96.52 0)
 			(effects
@@
 			)
 		)
-		(property "Description" "Power symbol creates a global label with name \"GND\" , ground"
+		(property "Description" ""
 			(at 176.53 63.5 0)
 			(effects
@@
 		(property "Mouser" "71-CRCW0603100RFKEAH"
 			(at 167.64 91.694 0)
-			(effects
-				(font
-					(size 1.27 1.27)
-				)
-				(hide yes)
-			)
-		)
-		(property "Sim.Pin" ""
-			(at 167.64 76.2 0)
 			(effects
 				(font
@@
 			)
 		)
-		(property "Description" "Power symbol creates a global label with name \"GND\" , ground"
+		(property "Description" ""
 			(at 143.51 118.11 0)
 			(effects
@@
 			)
 		)
-		(property "Sim.Pin" ""
-			(at 176.53 60.96 0)
-			(effects
-				(font
-					(size 1.27 1.27)
-				)
-				(hide yes)
-			)
-		)
 		(property "Manufacturer" "TDK"
 			(at 176.53 76.2 0)
@@
 			(effects
 				(font
+					(size 1.27 1.27)
+				)
+				(hide yes)
+			)
+		)
+		(property "Rating" "50V"
+			(at 176.53 83.82 0)
+			(effects
+				(font

Commit message: Update Library
Parts:
- C1001: symbol V2_Device:C_0603_0u1 -> V2_Capacitor:0603_0u1
- R1001: symbol V2_Device:R_0603_100R -> V2_Resistor:0603_100R
Changed lines of the file:
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@@
 	)
 	(symbol
-		(lib_id "V2_Device:R_0603_100R")
+		(lib_id "V2_Resistor:0603_100R")
 		(at 167.64 76.2 0)
 		(unit 1)
@@
 	)
 	(symbol
-		(lib_id "V2_Device:C_0603_0u1")
+		(lib_id "V2_Capacitor:0603_0u1")
 		(at 176.53 60.96 0)
 		(unit 1)

Commit message: Refresh
Other:
- note added: "PoE Passive +28V IEEE 802.3af Mode B"
- note removed: "PoE Passive +24V IEEE 802.3af Mode B"
Changed lines of the file:
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@@
 		(company "Socket")
 	)
-	(text "PoE Passive +24V\nIEEE 802.3af Mode B"
+	(text "PoE Passive +28V\nIEEE 802.3af Mode B"
 		(exclude_from_sim no)
 		(at 169.164 150.876 0)
@@
 		(dnp no)
 		(property "Reference" "R1001"
-			(at 172.72 74.93 0)
+			(at 172.466 75.184 0)
 			(effects
 				(font
@@
 		)
 		(property "Value" "100R"
-			(at 171.45 77.47 0)
-			(effects
-				(font
+			(at 171.958 77.216 0)
+			(effects
+				(font

Commit message: Replace diode
Other:
- title: V2 Link -> V2 drum

Commit message: Update
Parts:
- C1001: Id (none) -> Capacitor:${SYMBOL_NAME}
- J1001: Id (none) -> EtherCon:${SYMBOL_NAME}; Rating (none) -> CAT5e
- R1001: Id (none) -> Resistor:${SYMBOL_NAME}
- U1001: Id (none) -> RS485:${SYMBOL_NAME}; Rating (none) -> 20Mbps
Other:
- company: Socket -> Versio Duo
Changed lines of the file:
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@@
 	(title_block
 		(title "V2 drum")
-		(date "2026-03-30")
+		(date "2026-04-14")
 		(rev "2026-03-30")
-		(company "Socket")
+		(company "Versio Duo")
+		(comment 1 "Percussion Controller")
 	)
 	(text "PoE Passive +28V\nIEEE 802.3af Mode B"
@@
 		(in_pos_files yes)
 		(dnp no)
-		(property "Reference" "#PWR1001"
+		(property "Reference" "#PWR01002"
 			(at 154.94 62.23 0)
 			(hide yes)
@@
 			(project "drum"
 				(path "/6c8448b4-b04d-47e1-934e-e40cbe27a7be/2a03ea79-269e-4abf-833c-000ba0ff13d7"
-					(reference "#PWR1001")
+					(reference "#PWR01002")
 					(unit 1)
 				)
@@
 		(property "Manufacturer" "Texas Instruments"
 			(at 154.94 111.76 0)
+			(hide yes)
+			(show_name no)
+			(do_not_autoplace no)
+			(effects
+				(font
+					(size 1.27 1.27)
+				)
+			)
+		)
+		(property "Id" "RS485:${SYMBOL_NAME}"
+			(at 154.94 113.03 0)
+			(hide yes)
+			(show_name no)
+			(do_not_autoplace no)
+			(effects
+				(font
+					(size 1.27 1.27)
+				)
+			)
+		)
+		(property "Rating" "20Mbps"
+			(at 156.21 120.65 0)
 			(hide yes)
 			(show_name no)
@@
 			)
 		)
+		(property "Id" "EtherCon:${SYMBOL_NAME}"
+			(at 154.94 161.29 0)
+			(hide yes)
+			(show_name no)
+			(do_not_autoplace no)
+			(effects
+				(font
+					(size 1.27 1.27)
+				)
+			)
+		)
+		(property "Rating" "CAT5e"
+			(at 154.94 163.83 0)
+			(hide yes)
+			(show_name no)
+			(do_not_autoplace no)
+			(effects
+				(font
+					(size 1.27 1.27)
+				)
+			)
+		)
 		(pin "8"
 		)
@@
 		(in_pos_files yes)
 		(dnp no)
-		(property "Reference" "#PWR1003"
+		(property "Reference" "#PWR01003"
 			(at 154.94 102.87 0)
 			(hide yes)
@@
 			(project "drum"
 				(path "/6c8448b4-b04d-47e1-934e-e40cbe27a7be/2a03ea79-269e-4abf-833c-000ba0ff13d7"
-					(reference "#PWR1003")
+					(reference "#PWR01003")
 					(unit 1)
 				)
@@
 		(in_pos_files yes)
 		(dnp no)
-		(property "Reference" "#PWR1002"
+		(property "Reference" "#PWR01004"
 			(at 176.53 69.85 0)
 			(hide yes)
@@
 			(project "drum"
 				(path "/6c8448b4-b04d-47e1-934e-e40cbe27a7be/2a03ea79-269e-4abf-833c-000ba0ff13d7"
-					(reference "#PWR1002")
+					(reference "#PWR01004")
 					(unit 1)
 				)
@@
 			)
 		)
+		(property "Id" "Resistor:${SYMBOL_NAME}"
+			(at 167.64 90.17 0)
+			(hide yes)
+			(show_name no)
+			(do_not_autoplace no)
+			(effects
+				(font
+					(size 1.27 1.27)
+				)
+			)
+		)
 		(pin "1"
 		)
@@
 		(in_pos_files yes)
 		(dnp no)
-		(property "Reference" "#PWR1004"
+		(property "Reference" "#PWR01001"
 			(at 137.16 118.11 0)
 			(hide yes)
@@
 			(project "drum"
 				(path "/6c8448b4-b04d-47e1-934e-e40cbe27a7be/2a03ea79-269e-4abf-833c-000ba0ff13d7"
-					(reference "#PWR1004")
+					(reference "#PWR01001")
 					(unit 1)
 				)
@@
 			(hide yes)
 			(show_name no)
+			(do_not_autoplace no)
+			(effects
+				(font
+					(size 1.27 1.27)
+				)
+			)
+		)
+		(property "Id" "Capacitor:${SYMBOL_NAME}"
+			(at 176.53 76.2 0)
+			(hide yes)
+			(show_name no)
