File: StepperDriver.kicad_sch (KiCad schematic)
At the start: 18 parts, among them J701 Conn_01x01, J702 Conn_01x01, J703 Conn_01x01, J704 Conn_01x01, U701 TMC2130-LA

Commit message: Update parts
Parts:
- C701, C708: footprint Capacitor_SMD:C_0603_1608Metric -> V2_Capacitor_SMD:C_0603; symbol Device:C_Small -> V2_Device:C_0603_0u1; Manufacturer (none) -> TDK; Mouser (none) -> 810-CGA3E2X7R1H104MA; Product (none) -> CGA3E2X7R1H104M080AA
- C702, C703: footprint Capacitor_SMD:CP_Elec_6.3x5.8 -> V2_Capacitor_SMD:CP_Elec_6.3x7.7; symbol Device:C_Polarized_Small -> V2_Device:C_Polarized_6.3x7.7_100u; Manufacturer (none) -> Panasonic; Mouser (none) -> 667-EEE-FKV101XAL; Product (none) -> EEE-FKV101XAL; Rating (none) -> 35V
- C704, C705: footprint Capacitor_SMD:C_1210_3225Metric -> V2_Capacitor_SMD:C_1210; symbol Device:C_Small -> V2_Device:C_1210_10u; Manufacturer (none) -> TDK; Mouser (none) -> 810-CNA6P1X7R1H106K2; Product (none) -> CNA6P1X7R1H106K250AE; Rating (none) -> 50V; Voltage (none) -> 50V
- C706: footprint Capacitor_SMD:C_0603_1608Metric -> V2_Capacitor_SMD:C_0603; symbol Device:C_Small -> V2_Device:C_0603_4u7; Manufacturer (none) -> YAGEO; Mouser (none) -> 603-CC603KRX5R6BB475; Product (none) -> CC0603KRX5R6BB475
- C707: value 0u470 -> 0u47; footprint Capacitor_SMD:C_0603_1608Metric -> V2_Capacitor_SMD:C_0603; symbol Device:C_Small -> V2_Device:C_0603_0u47; Manufacturer (none) -> YAGEO; Mouser (none) -> 603-CC0603JR6BB474; Product (none) -> CC0603JRX7R6BB474
- C709: footprint Capacitor_SMD:C_0603_1608Metric -> V2_Capacitor_SMD:C_0603; symbol Device:C_Small -> V2_Device:C_0603_0u022; Manufacturer (none) -> YAGEO; Mouser (none) -> 603-CC603KPX7R9BB223; Product (none) -> CC0603KPX7R9BB223
- D701: LCSC (none) -> C965555; Manufacturer (none) -> Worldsemi; Product (none) -> WS2812B-2020
- J701, J702, J703, J704: value Conn_01x01 -> WAGO 2065-100; Manufacturer (none) -> WAGO; Product (none) -> 2065-100/998-403
- R701: footprint Resistor_SMD:R_0603_1608Metric -> V2_Resistor_SMD:R_0603; symbol Device:R_Small -> V2_Device:R_0603_2R2; Manufacturer (none) -> Vishay; Mouser (none) -> 71-RCS06032R20JNEA; Product (none) -> RCS06032R20JNEA; Rating (none) -> 500mW
- R702, R703: footprint Resistor_SMD:R_0805_2012Metric -> V2_Resistor_SMD:R_0805; symbol Device:R_Small -> V2_Device:R_0805_0R11; Manufacturer (none) -> Panasonic; Mouser (none) -> 667-ERJ-6DSFR11V; Product (none) -> ERJ-6DSFR11V; Rating (none) -> 500mW
- U701: LCSC (none) -> C915795; Manufacturer (none) -> Analog Devices; Product (none) -> TMC2130-LA

Commit message: Update library
Parts:
- C701, C708: Rating (none) -> 50V
- C704, C705: Voltage 50V -> (none)
Connections:
- net +24V renamed +28V
Changed lines of the file:
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@@
-			)
-		)
-		(property "Sim.Pin" ""
-			(at 158.75 49.53 0)
-			(effects
-				(font
-					(size 1.27 1.27)
-				)
-				(hide yes)
 			)
 		)
@@
 			)
 		)
-		(property "Voltage" "50V"
-			(at 158.75 69.85 0)
-			(effects
-				(font
-					(size 1.27 1.27)
-				)
-				(hide yes)
-			)
-		)
 		(pin "1"
 		)
@@
 			)
 		)
-		(property "Sim.Pin" ""
-			(at 110.49 81.28 0)
-			(effects
-				(font
-					(size 1.27 1.27)
-				)
-				(hide yes)
-			)
-		)
 		(property "Product" "CC0603KRX5R6BB475"
 			(at 110.49 99.06 0)
@@
 	)
 	(symbol
-		(lib_id "V2_power:+24V")
+		(lib_id "V2_power:+28V")
 		(at 139.7 88.9 90)
 		(unit 1)
@@
 			)
 		)
-		(property "Value" "+24V"
+		(property "Value" "+28V"
 			(at 135.89 88.8999 90)
 			(effects
@@
 			)
 		)
-		(property "Description" "Power symbol creates a global label with name \"+24V\""
+		(property "Description" ""
 			(at 139.7 88.9 0)
 			(effects
@@
 			)
 		)
-		(property "Sim.Pin" ""
-			(at 175.26 91.44 0)
-			(effects
-				(font
-					(size 1.27 1.27)
-				)
-				(hide yes)
-			)
-		)
 		(property "Product" "CC0603KPX7R9BB223"
 			(at 175.26 109.22 0)
@@
 			)
 		)
-		(property "Sim.Pin" ""
-			(at 170.18 49.53 0)
-			(effects
-				(font
-					(size 1.27 1.27)
-				)
-				(hide yes)
-			)
-		)
 		(property "Product" "CNA6P1X7R1H106K250AE"
 			(at 170.18 67.31 0)
@@
 		(property "Manufacturer" "TDK"
 			(at 170.18 64.77 0)
-			(effects
-				(font
-					(size 1.27 1.27)
-				)
-				(hide yes)
-			)
-		)
-		(property "Voltage" "50V"
-			(at 170.18 69.85 0)
 			(effects
 				(font
@@
 			)
 		)
-		(property "Description" "Power symbol creates a global label with name \"GND\" , ground"
+		(property "Description" ""
 			(at 191.77 129.54 0)
 			(effects
@@
 			)
 		)
-		(property "Sim.Pin" ""
-			(at 157.48 160.02 0)
-			(effects
-				(font
-					(size 1.27 1.27)
-				)
-				(hide yes)
-			)
-		)
 		(pin "1"
 		)
@@
 			)
 		)
-		(property "Sim.Pin" ""
-			(at 124.46 49.53 0)
-			(effects
-				(font
-					(size 1.27 1.27)
-				)
-				(hide yes)
-			)
-		)
 		(property "Manufacturer" "TDK"
 			(at 124.46 64.77 0)
@@
 		(property "Product" "CGA3E2X7R1H104M080AA"
 			(at 124.46 67.31 0)
+			(effects
+				(font
+					(size 1.27 1.27)
+				)
+				(hide yes)
+			)
+		)
+		(property "Rating" "50V"
+			(at 124.46 72.39 0)
 			(effects
 				(font
@@
 			)
 		)
-		(property "Description" "Power symbol creates a global label with name \"GND\" , ground"
+		(property "Description" ""
 			(at 175.26 139.7 0)
 			(effects
@@
 			)
 		)
-		(property "Description" "Power symbol creates a global label with name \"+5V\""
+		(property "Description" ""
 			(at 165.1 156.21 0)
 			(effects
@@
 			)
 		)
-		(property "Description" "Power symbol creates a global label with name \"GND\" , ground"
+		(property "Description" ""
 			(at 191.77 127 0)
 			(effects
@@
 			)
 		)
-		(property "Sim.Pin" ""
-			(at 189.23 127 90)
-			(effects
-				(font
-					(size 1.27 1.27)
-				)
-				(hide yes)
-			)
-		)
 		(property "Product" "ERJ-6DSFR11V"
 			(at 207.01 127 0)
@@
 			)
 		)
-		(property "Description" "Power symbol creates a global label with name \"GND\" , ground"
+		(property "Description" ""
 			(at 124.46 52.07 0)
 			(effects
@@
 			)
 		)
-		(property "Sim.Pin" ""
-			(at 139.7 86.36 0)
-			(effects
-				(font
-					(size 1.27 1.27)
-				)
-				(hide yes)
-			)
-		)
 		(property "Manufacturer" "TDK"
 			(at 139.7 101.6 0)
@@
 			)
 		)
+		(property "Rating" "50V"
+			(at 139.7 109.22 0)
+			(effects
+				(font
+					(size 1.27 1.27)
+				)
+				(hide yes)
+			)
+		)
 		(pin "1"
 		)
@@
 			)
 		)
-		(property "Description" "Power symbol creates a global label with name \"GND\" , ground"
+		(property "Description" ""
 			(at 170.18 52.07 0)
 			(effects
@@
 			)
 		)
-		(property "Description" "Power symbol creates a global label with name \"GND\" , ground"
+		(property "Description" ""
 			(at 139.7 104.14 0)
 			(effects
@@
 			)
 		)
-		(property "Description" "Power symbol creates a global label with name \"+3V3\""
+		(property "Description" ""
 			(at 139.7 81.28 0)
 			(effects
@@
 			)
 		)
-		(property "Description" "Power symbol creates a global label with name \"+3V3\""
+		(property "Description" ""
 			(at 124.46 46.99 0)
 			(effects
@@
 	)
 	(symbol
-		(lib_id "V2_power:+24V")
+		(lib_id "V2_power:+28V")
 		(at 139.7 91.44 90)
 		(unit 1)
@@
 			)
 		)
-		(property "Value" "+24V"
+		(property "Value" "+28V"
 			(at 135.89 91.4399 90)
 			(effects
@@
 			)
 		)
-		(property "Description" "Power symbol creates a global label with name \"+24V\""
+		(property "Description" ""
 			(at 139.7 91.44 0)
 			(effects
@@
 			)
 		)
-		(property "Description" "Power symbol creates a global label with name \"GND\" , ground"
+		(property "Description" ""
 			(at 123.19 83.82 0)
 			(effects
@@
 			)
 		)
-		(property "Sim.Pin" ""
-			(at 134.62 49.53 0)
-			(effects
-				(font
-					(size 1.27 1.27)
-				)
-				(hide yes)
-			)
-		)
 		(property "Product" "EEE-FKV101XAL"
 			(at 134.62 69.85 0)
@@
 		(property "Mouser" "667-EEE-FKV101XAL"
 			(at 147.32 70.104 0)
-			(effects
-				(font
-					(size 1.27 1.27)
-				)
-				(hide yes)
-			)
-		)
-		(property "Sim.Pin" ""
-			(at 147.32 49.53 0)
 			(effects
 				(font
@@
 			)
 		)
-		(property "Sim.Pin" ""
-			(at 189.23 83.82 0)
-			(effects
-				(font
-					(size 1.27 1.27)
-				)
-				(hide yes)
-			)
-		)
 		(pin "1"
 		)
@@
 			)
 		)
-		(property "Sim.Pin" ""
-			(at 189.23 81.28 0)
-			(effects
-				(font
-					(size 1.27 1.27)
-				)
-				(hide yes)
-			)
-		)
 		(pin "1"
 		)
@@
 			)
 		)
-		(property "Description" "Power symbol creates a global label with name \"GND\" , ground"
+		(property "Description" ""
 			(at 139.7 106.68 0)
 			(effects
@@
 			)
 		)
-		(property "Description" "Power symbol creates a global label with name \"GND\" , ground"
+		(property "Description" ""
 			(at 110.49 83.82 0)
 			(effects
@@
 		(property "Mouser" "71-RCS06032R20JNEA"
 			(at 132.334 78.74 0)
-			(effects
-				(font
-					(size 1.27 1.27)
-				)
-				(hide yes)
-			)
-		)
-		(property "Sim.Pin" ""
-			(at 116.84 78.74 90)
 			(effects
 				(font
@@
 			)
 		)
-		(property "Sim.Pin" ""
-			(at 157.48 106.68 0)
-			(effects
-				(font
-					(size 1.27 1.27)
-				)
-				(hide yes)
-			)
-		)
 		(pin "13"
 		)
@@
 			)
 		)
-		(property "Sim.Pin" ""
-			(at 189.23 76.2 0)
-			(effects
-				(font
-					(size 1.27 1.27)
-				)
-				(hide yes)
-			)
-		)
 		(pin "1"
 		)
@@
 			)
 		)
-		(property "Sim.Pin" ""
-			(at 189.23 129.54 90)
-			(effects
-				(font
-					(size 1.27 1.27)
-				)
-				(hide yes)
-			)
-		)
 		(property "Product" "ERJ-6DSFR11V"
 			(at 207.01 129.54 0)
@@
 	)
 	(symbol
-		(lib_id "V2_power:+24V")
+		(lib_id "V2_power:+28V")
 		(at 170.18 46.99 0)
 		(unit 1)
@@
 			)
 		)
-		(property "Value" "+24V"
+		(property "Value" "+28V"
 			(at 170.18 41.91 0)
 			(effects
@@
 			)
 		)
-		(property "Description" "Power symbol creates a global label with name \"+24V\""
+		(property "Description" ""
 			(at 170.18 46.99 0)
 			(effects
@@
 		(property "Mouser" "603-CC0603JR6BB474"
 			(at 123.19 98.298 0)
-			(effects
-				(font
-					(size 1.27 1.27)
-				)
-				(hide yes)
-			)
-		)
-		(property "Sim.Pin" ""
-			(at 123.19 81.28 0)
 			(effects
 				(font
@@
 			)
 		)
-		(property "Description" "Power symbol creates a global label with name \"GND\" , ground"
+		(property "Description" ""
 			(at 139.7 124.46 0)
 			(effects
@@
 			)
 		)
-		(property "Sim.Pin" ""
-			(at 189.23 73.66 0)
-			(effects
-				(font
-					(size 1.27 1.27)
-				)
-				(hide yes)
-			)
-		)
 		(pin "1"
 		)
@@
 			)
 		)
-		(property "Description" "Power symbol creates a global label with name \"GND\" , ground"
+		(property "Description" ""
 			(at 165.1 161.29 0)
 			(effects

Commit message: Update library
Parts:
- U701: footprint V2_Driver_Stepper:QFN36-5X6 -> V2_Package_DFN_QFN:QFN36-5X6
Changed lines of the file:
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@@
 			)
 		)
-		(property "Footprint" "V2_Driver_Stepper:QFN36-5X6"
+		(property "Footprint" "V2_Package_DFN_QFN:QFN36-5X6"
 			(at 158.75 150.114 0)
 			(effects

Commit message: Update Library
Parts:
- C701, C708: symbol V2_Device:C_0603_0u1 -> V2_Capacitor:0603_0u1
- C702, C703: symbol V2_Device:C_Polarized_6.3x7.7_100u -> V2_Capacitor:Polarized_6.3x7.7_100u
- C704, C705: symbol V2_Device:C_1210_10u -> V2_Capacitor:1210_10u
- C706: symbol V2_Device:C_0603_4u7 -> V2_Capacitor:0603_4u7
- C707: symbol V2_Device:C_0603_0u47 -> V2_Capacitor:0603_0u47
- C709: symbol V2_Device:C_0603_0u022 -> V2_Capacitor:0603_0u022
- R701: symbol V2_Device:R_0603_2R2 -> V2_Resistor:0603_2R2
- R702, R703: symbol V2_Device:R_0805_0R11 -> V2_Resistor:0805_0R11
Changed lines of the file:
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@@
 	)
 	(symbol
-		(lib_id "V2_Device:C_1210_10u")
+		(lib_id "V2_Capacitor:1210_10u")
 		(at 158.75 49.53 0)
 		(unit 1)
@@
 	)
 	(symbol
-		(lib_id "V2_Device:C_0603_4u7")
+		(lib_id "V2_Capacitor:0603_4u7")
 		(at 110.49 81.28 0)
 		(unit 1)
@@
 	)
 	(symbol
-		(lib_id "V2_Device:C_0603_0u022")
+		(lib_id "V2_Capacitor:0603_0u022")
 		(at 175.26 91.44 0)
 		(unit 1)
@@
 	)
 	(symbol
-		(lib_id "V2_Device:C_1210_10u")
+		(lib_id "V2_Capacitor:1210_10u")
 		(at 170.18 49.53 0)
 		(unit 1)
@@
 	)
 	(symbol
-		(lib_id "V2_Device:C_0603_0u1")
+		(lib_id "V2_Capacitor:0603_0u1")
 		(at 124.46 49.53 0)
 		(unit 1)
@@
 	)
 	(symbol
-		(lib_id "V2_Device:R_0805_0R11")
+		(lib_id "V2_Resistor:0805_0R11")
 		(at 189.23 127 90)
 		(unit 1)
@@
 	)
 	(symbol
-		(lib_id "V2_Device:C_0603_0u1")
+		(lib_id "V2_Capacitor:0603_0u1")
 		(at 139.7 86.36 0)
 		(unit 1)
@@
 	)
 	(symbol
-		(lib_id "V2_Device:C_Polarized_6.3x7.7_100u")
+		(lib_id "V2_Capacitor:Polarized_6.3x7.7_100u")
 		(at 134.62 49.53 0)
 		(unit 1)
@@
 	)
 	(symbol
-		(lib_id "V2_Device:C_Polarized_6.3x7.7_100u")
+		(lib_id "V2_Capacitor:Polarized_6.3x7.7_100u")
 		(at 147.32 49.53 0)
 		(unit 1)
@@
 	)
 	(symbol
-		(lib_id "V2_Device:R_0603_2R2")
+		(lib_id "V2_Resistor:0603_2R2")
 		(at 116.84 78.74 90)
 		(unit 1)
@@
 	)
 	(symbol
-		(lib_id "V2_Device:R_0805_0R11")
+		(lib_id "V2_Resistor:0805_0R11")
 		(at 189.23 129.54 90)
 		(unit 1)
@@
 	)
 	(symbol
-		(lib_id "V2_Device:C_0603_0u47")
+		(lib_id "V2_Capacitor:0603_0u47")
 		(at 123.19 81.28 0)
 		(unit 1)

Commit message: Replace diode
Parts:
- C704, C705: Mouser 810-CNA6P1X7R1H106K2 -> 810-CNC6P1X7R1H106K2; Product CNA6P1X7R1H106K250AE -> CNC6P1X7R1H106K250AE
- U701: footprint V2_Package_DFN_QFN:QFN36-5X6 -> V2_Package_DFN_QFN:QFN-36-5X6
Changed lines of the file:
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@@
 			)
 		)
-		(property "Description" "Unpolarized capacitor, small symbol"
+		(property "Description" ""
 			(at 158.75 62.992 0)
 			(effects
@@
 			)
 		)
-		(property "Mouser" "810-CNA6P1X7R1H106K2"
+		(property "Mouser" "810-CNC6P1X7R1H106K2"
 			(at 158.75 66.04 0)
 			(effects
@@
 			)
 		)
-		(property "Product" "CNA6P1X7R1H106K250AE"
+		(property "Product" "CNC6P1X7R1H106K250AE"
 			(at 158.75 67.31 0)
 			(effects
@@
 			)
 		)
-		(property "Description" "Unpolarized capacitor, small symbol"
+		(property "Description" ""
 			(at 110.49 94.742 0)
 			(effects
@@
 		(dnp no)
 		(fields_autoplaced yes)
-		(property "Reference" "#PWR0708"
+		(property "Reference" "#PWR708"
 			(at 143.51 88.9 0)
 			(effects
@@
 			(project "hihat-1"
 				(path "/6c8448b4-b04d-47e1-934e-e40cbe27a7be/3587b23e-cce2-48a9-8cab-0ba93735c629"
-					(reference "#PWR0708")
+					(reference "#PWR708")
 					(unit 1)
 				)
@@
 			)
 		)
-		(property "Description" "Unpolarized capacitor, small symbol"
+		(property "Description" ""
 			(at 175.26 104.902 0)
 			(effects
@@
 			)
 		)
-		(property "Description" "Unpolarized capacitor, small symbol"
+		(property "Description" ""
 			(at 170.18 62.992 0)
 			(effects
@@
 			)
 		)
-		(property "Mouser" "810-CNA6P1X7R1H106K2"
+		(property "Mouser" "810-CNC6P1X7R1H106K2"
 			(at 170.18 66.04 0)
 			(effects
@@
 			)
 		)
-		(property "Product" "CNA6P1X7R1H106K250AE"
+		(property "Product" "CNC6P1X7R1H106K250AE"
 			(at 170.18 67.31 0)
 			(effects
@@
 		(dnp no)
 		(fields_autoplaced yes)
-		(property "Reference" "#PWR0714"
+		(property "Reference" "#PWR714"
 			(at 198.12 129.54 0)
 			(effects
@@
 			(project "hihat-1"
 				(path "/6c8448b4-b04d-47e1-934e-e40cbe27a7be/3587b23e-cce2-48a9-8cab-0ba93735c629"
-					(reference "#PWR0714")
+					(reference "#PWR714")
 					(unit 1)
 				)
@@
 			)
 		)
-		(property "Description" "Unpolarized capacitor, small symbol"
+		(property "Description" ""
 			(at 124.46 62.992 0)
 			(effects
@@
 		(dnp no)
 		(fields_autoplaced yes)
-		(property "Reference" "#PWR0715"
+		(property "Reference" "#PWR715"
 			(at 181.61 139.7 0)
 			(effects
@@
 			(project "hihat-1"
 				(path "/6c8448b4-b04d-47e1-934e-e40cbe27a7be/3587b23e-cce2-48a9-8cab-0ba93735c629"
-					(reference "#PWR0715")
+					(reference "#PWR715")
 					(unit 1)
 				)
@@
 		(on_board yes)
 		(dnp no)
-		(property "Reference" "#PWR0716"
+		(property "Reference" "#PWR716"
 			(at 161.29 156.21 0)
 			(effects
@@
 			(project "hihat-1"
 				(path "/6c8448b4-b04d-47e1-934e-e40cbe27a7be/3587b23e-cce2-48a9-8cab-0ba93735c629"
-					(reference "#PWR0716")
+					(reference "#PWR716")
 					(unit 1)
 				)
@@
 		(dnp no)
 		(fields_autoplaced yes)
-		(property "Reference" "#PWR0713"
+		(property "Reference" "#PWR713"
 			(at 198.12 127 0)
 			(effects
@@
 			(project "hihat-1"
 				(path "/6c8448b4-b04d-47e1-934e-e40cbe27a7be/3587b23e-cce2-48a9-8cab-0ba93735c629"
-					(reference "#PWR0713")
+					(reference "#PWR713")
 					(unit 1)
 				)
@@
 			)
 		)
-		(property "Description" "Resistor, small symbol"
+		(property "Description" ""
 			(at 201.422 127 0)
 			(effects
@@
 		(on_board yes)
 		(dnp no)
-		(property "Reference" "#PWR0703"
+		(property "Reference" "#PWR703"
 			(at 124.46 58.42 0)
 			(effects
@@
 			(project "hihat-1"
 				(path "/6c8448b4-b04d-47e1-934e-e40cbe27a7be/3587b23e-cce2-48a9-8cab-0ba93735c629"
-					(reference "#PWR0703")
+					(reference "#PWR703")
 					(unit 1)
 				)
@@
 			)
 		)
-		(property "Description" "Unpolarized capacitor, small symbol"
+		(property "Description" ""
 			(at 139.7 99.822 0)
 			(effects
@@
 		(on_board yes)
 		(dnp no)
-		(property "Reference" "#PWR0704"
+		(property "Reference" "#PWR704"
 			(at 170.18 58.42 0)
 			(effects
@@
 			(project "hihat-1"
 				(path "/6c8448b4-b04d-47e1-934e-e40cbe27a7be/3587b23e-cce2-48a9-8cab-0ba93735c629"
-					(reference "#PWR0704")
+					(reference "#PWR704")
 					(unit 1)
 				)
@@
 		(dnp no)
 		(fields_autoplaced yes)
-		(property "Reference" "#PWR0710"
+		(property "Reference" "#PWR710"
 			(at 133.35 104.14 0)
 			(effects
@@
 			(project "hihat-1"
 				(path "/6c8448b4-b04d-47e1-934e-e40cbe27a7be/3587b23e-cce2-48a9-8cab-0ba93735c629"
-					(reference "#PWR0710")
+					(reference "#PWR710")
 					(unit 1)
 				)
@@
 		(dnp no)
 		(fields_autoplaced yes)
-		(property "Reference" "#PWR0705"
+		(property "Reference" "#PWR705"
 			(at 143.51 81.28 0)
 			(effects
@@
 			(project "hihat-1"
 				(path "/6c8448b4-b04d-47e1-934e-e40cbe27a7be/3587b23e-cce2-48a9-8cab-0ba93735c629"
-					(reference "#PWR0705")
+					(reference "#PWR705")
 					(unit 1)
 				)
@@
 		(dnp no)
 		(fields_autoplaced yes)
-		(property "Reference" "#PWR0701"
+		(property "Reference" "#PWR701"
 			(at 124.46 50.8 0)
 			(effects
@@
 			(project "hihat-1"
 				(path "/6c8448b4-b04d-47e1-934e-e40cbe27a7be/3587b23e-cce2-48a9-8cab-0ba93735c629"
-					(reference "#PWR0701")
+					(reference "#PWR701")
 					(unit 1)
 				)
@@
 		(dnp no)
 		(fields_autoplaced yes)
-		(property "Reference" "#PWR0709"
+		(property "Reference" "#PWR709"
 			(at 143.51 91.44 0)
 			(effects
@@
 			(project "hihat-1"
 				(path "/6c8448b4-b04d-47e1-934e-e40cbe27a7be/3587b23e-cce2-48a9-8cab-0ba93735c629"
-					(reference "#PWR0709")
+					(reference "#PWR709")
 					(unit 1)
 				)
@@
 		(dnp no)
 		(fields_autoplaced yes)
-		(property "Reference" "#PWR0707"
+		(property "Reference" "#PWR707"
 			(at 123.19 90.17 0)
 			(effects
@@
 			(project "hihat-1"
 				(path "/6c8448b4-b04d-47e1-934e-e40cbe27a7be/3587b23e-cce2-48a9-8cab-0ba93735c629"
-					(reference "#PWR0707")
+					(reference "#PWR707")
 					(unit 1)
 				)
@@
 			)
 		)
-		(property "Description" "Polarized capacitor, small symbol"
+		(property "Description" ""
 			(at 134.62 62.738 0)
 			(effects
@@
 			)
 		)
-		(property "Description" "Polarized capacitor, small symbol"
+		(property "Description" ""
 			(at 147.32 62.738 0)
 			(effects
@@
 		(dnp no)
 		(fields_autoplaced yes)
-		(property "Reference" "#PWR0711"
+		(property "Reference" "#PWR711"
 			(at 133.35 106.68 0)
 			(effects
@@
 			(project "hihat-1"
 				(path "/6c8448b4-b04d-47e1-934e-e40cbe27a7be/3587b23e-cce2-48a9-8cab-0ba93735c629"
-					(reference "#PWR0711")
+					(reference "#PWR711")
 					(unit 1)
 				)
@@
 		(dnp no)
 		(fields_autoplaced yes)
-		(property "Reference" "#PWR0706"
+		(property "Reference" "#PWR706"
 			(at 110.49 90.17 0)
 			(effects
@@
 			(project "hihat-1"
 				(path "/6c8448b4-b04d-47e1-934e-e40cbe27a7be/3587b23e-cce2-48a9-8cab-0ba93735c629"
-					(reference "#PWR0706")
+					(reference "#PWR706")
 					(unit 1)
 				)
@@
 			)
 		)
-		(property "Description" "Resistor, small symbol"
+		(property "Description" ""
 			(at 129.032 78.74 0)
 			(effects
@@
 			)
 		)
-		(property "Footprint" "V2_Package_DFN_QFN:QFN36-5X6"
+		(property "Footprint" "V2_Package_DFN_QFN:QFN-36-5X6"
 			(at 158.75 150.114 0)
 			(effects
@@
 			)
 		)
-		(property "Description" "Resistor, small symbol"
+		(property "Description" ""
 			(at 201.422 129.54 0)
 			(effects
@@
 		(dnp no)
 		(fields_autoplaced yes)
-		(property "Reference" "#PWR0702"
+		(property "Reference" "#PWR702"
 			(at 170.18 50.8 0)
 			(effects
@@
 			(project "hihat-1"
 				(path "/6c8448b4-b04d-47e1-934e-e40cbe27a7be/3587b23e-cce2-48a9-8cab-0ba93735c629"
-					(reference "#PWR0702")
+					(reference "#PWR702")
 					(unit 1)
 				)
@@
 			)
 		)
-		(property "Description" "Unpolarized capacitor, small symbol"
+		(property "Description" ""
 			(at 123.19 94.742 0)
 			(effects
@@
 		(dnp no)
 		(fields_autoplaced yes)
-		(property "Reference" "#PWR0712"
+		(property "Reference" "#PWR712"
 			(at 133.35 124.46 0)
 			(effects
@@
 			(project "hihat-1"
 				(path "/6c8448b4-b04d-47e1-934e-e40cbe27a7be/3587b23e-cce2-48a9-8cab-0ba93735c629"
-					(reference "#PWR0712")
+					(reference "#PWR712")
 					(unit 1)
 				)
@@
 		(on_board yes)
 		(dnp no)
-		(property "Reference" "#PWR0717"
+		(property "Reference" "#PWR717"
 			(at 171.45 161.29 0)
 			(effects
@@
 			(project "hihat-1"
 				(path "/6c8448b4-b04d-47e1-934e-e40cbe27a7be/3587b23e-cce2-48a9-8cab-0ba93735c629"
-					(reference "#PWR0717")
+					(reference "#PWR717")
 					(unit 1)
 				)
@@
 		(on_board yes)
 		(dnp no)
-		(property "Reference" "#FLG0701"
+		(property "Reference" "#FLG701"
 			(at 124.46 76.835 0)
 			(effects
@@
 			(project "hihat-1"
 				(path "/6c8448b4-b04d-47e1-934e-e40cbe27a7be/3587b23e-cce2-48a9-8cab-0ba93735c629"
-					(reference "#FLG0701")
-					(unit 1)
-				)
+					(reference "#FLG701")
+					(unit 1)
+				)

Commit message: Replace diode
Other:
- title: Stepper Driver -> V2 drum

Commit message: Update
Parts:
- C701: renamed from C706; Id (none) -> Capacitor:${SYMBOL_NAME}; Rating (none) -> 10V
- C702: renamed from C707; Id (none) -> Capacitor:${SYMBOL_NAME}; Manufacturer YAGEO -> TDK; Mouser 603-CC0603JR6BB474 -> 810-CGA3E3X7R1H474KB; Product CC0603JRX7R6BB474 -> CGA3E3X7R1H474K080AB; Rating (none) -> 50V
- C703: renamed from C701; Id (none) -> Capacitor:${SYMBOL_NAME}
- C704: renamed from C702; Id (none) -> Capacitor:${SYMBOL_NAME}
- C705: renamed from C708; Id (none) -> Capacitor:${SYMBOL_NAME}
- C706: renamed from C703; Id (none) -> Capacitor:${SYMBOL_NAME}
- C707: renamed from C704; Id (none) -> Capacitor:${SYMBOL_NAME}
- C708: renamed from C705; Id (none) -> Capacitor:${SYMBOL_NAME}
- C709: Id (none) -> Capacitor:${SYMBOL_NAME}; Rating (none) -> 50V
- D701: Id (none) -> LED:${SYMBOL_NAME}; Rating (none) -> 15mA
- J701, J702, J703, J704: Id (none) -> WAGO:${SYMBOL_NAME}; Rating (none) -> 9A
- R701, R702, R703: Id (none) -> Resistor:${SYMBOL_NAME}
- U701: Id (none) -> Stepper:${SYMBOL_NAME}; Rating (none) -> 2A
