File: PowerSwitch.kicad_sch (KiCad schematic)
At the start: 16 parts, among them U401 BTT6010

Commit message: Refresh
Connections:
- net Power renamed +VPWM
Changed lines of the file:
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@@
 	(title_block
 		(title "V2 drum")
-		(date "2026-06-20")
+		(date "2026-08-28")
 		(rev "2026-05-25")
 		(company "Versio Duo")
@@
 		)
 	)
-	(hierarchical_label "Power"
+	(hierarchical_label "+VPWM"
 		(shape output)
 		(at 203.2 116.84 0)
@@
 		(in_pos_files no)
 		(dnp no)
-		(property "Reference" "#PWR409"
+		(property "Reference" "#PWR0409"
 			(at 166.37 48.26 0)
 			(hide yes)
@@
 			(project "drum"
 				(path "/6c8448b4-b04d-47e1-934e-e40cbe27a7be/ba748654-beb9-4861-aa35-c19e08caaf2e"
-					(reference "#PWR409")
+					(reference "#PWR0409")
 					(unit 1)
 				)
@@
 		(in_pos_files yes)
 		(dnp no)
-		(property "Reference" "#PWR414"
+		(property "Reference" "#PWR0414"
 			(at 191.77 63.5 0)
 			(hide yes)
@@
 			(project "drum"
 				(path "/6c8448b4-b04d-47e1-934e-e40cbe27a7be/ba748654-beb9-4861-aa35-c19e08caaf2e"
-					(reference "#PWR414")
+					(reference "#PWR0414")
 					(unit 1)
 				)
@@
 		(in_pos_files yes)
 		(dnp no)
-		(property "Reference" "#PWR403"
+		(property "Reference" "#PWR0403"
 			(at 127 143.51 0)
 			(hide yes)
@@
 			(project "drum"
 				(path "/6c8448b4-b04d-47e1-934e-e40cbe27a7be/ba748654-beb9-4861-aa35-c19e08caaf2e"
-					(reference "#PWR403")
+					(reference "#PWR0403")
 					(unit 1)
 				)
@@
 		(in_pos_files yes)
 		(dnp no)
-		(property "Reference" "#PWR412"
+		(property "Reference" "#PWR0412"
 			(at 184.15 128.27 0)
 			(hide yes)
@@
 			(project "drum"
 				(path "/6c8448b4-b04d-47e1-934e-e40cbe27a7be/ba748654-beb9-4861-aa35-c19e08caaf2e"
-					(reference "#PWR412")
+					(reference "#PWR0412")
 					(unit 1)
 				)
@@
 		(in_pos_files yes)
 		(dnp no)
-		(property "Reference" "#PWR401"
+		(property "Reference" "#PWR0401"
 			(at 114.3 116.84 0)
 			(hide yes)
@@
 			(project "drum"
 				(path "/6c8448b4-b04d-47e1-934e-e40cbe27a7be/ba748654-beb9-4861-aa35-c19e08caaf2e"
-					(reference "#PWR401")
+					(reference "#PWR0401")
 					(unit 1)
 				)
@@
 		(in_pos_files yes)
 		(dnp no)
-		(property "Reference" "#PWR413"
+		(property "Reference" "#PWR0413"
 			(at 186.69 111.76 0)
 			(hide yes)
@@
 			(project "drum"
 				(path "/6c8448b4-b04d-47e1-934e-e40cbe27a7be/ba748654-beb9-4861-aa35-c19e08caaf2e"
-					(reference "#PWR413")
+					(reference "#PWR0413")
 					(unit 1)
 				)
@@
 		(in_pos_files yes)
 		(dnp no)
-		(property "Reference" "#PWR411"
+		(property "Reference" "#PWR0411"
 			(at 166.37 96.52 0)
 			(hide yes)
@@
 			(project "drum"
 				(path "/6c8448b4-b04d-47e1-934e-e40cbe27a7be/ba748654-beb9-4861-aa35-c19e08caaf2e"
-					(reference "#PWR411")
+					(reference "#PWR0411")
 					(unit 1)
 				)
@@
 		(in_pos_files yes)
 		(dnp no)
-		(property "Reference" "#PWR407"
+		(property "Reference" "#PWR0407"
 			(at 162.56 132.08 0)
 			(hide yes)
@@
 			(project "drum"
 				(path "/6c8448b4-b04d-47e1-934e-e40cbe27a7be/ba748654-beb9-4861-aa35-c19e08caaf2e"
-					(reference "#PWR407")
+					(reference "#PWR0407")
 					(unit 1)
 				)
@@
 		(in_pos_files no)
 		(dnp no)
-		(property "Reference" "#PWR404"
+		(property "Reference" "#PWR0404"
 			(at 139.7 116.84 0)
 			(hide yes)
@@
 			(project "drum"
 				(path "/6c8448b4-b04d-47e1-934e-e40cbe27a7be/ba748654-beb9-4861-aa35-c19e08caaf2e"
-					(reference "#PWR404")
+					(reference "#PWR0404")
 					(unit 1)
 				)
@@
 		(in_pos_files yes)
 		(dnp no)
-		(property "Reference" "#PWR406"
+		(property "Reference" "#PWR0406"
 			(at 135.89 143.51 0)
 			(hide yes)
@@
 			(project "drum"
 				(path "/6c8448b4-b04d-47e1-934e-e40cbe27a7be/ba748654-beb9-4861-aa35-c19e08caaf2e"
-					(reference "#PWR406")
+					(reference "#PWR0406")
 					(unit 1)
 				)
@@
 		(in_pos_files yes)
 		(dnp no)
-		(property "Reference" "#PWR410"
+		(property "Reference" "#PWR0410"
 			(at 166.37 63.5 0)
 			(hide yes)
@@
 			(project "drum"
 				(path "/6c8448b4-b04d-47e1-934e-e40cbe27a7be/ba748654-beb9-4861-aa35-c19e08caaf2e"
-					(reference "#PWR410")
+					(reference "#PWR0410")
 					(unit 1)
 				)
@@
 		(in_pos_files yes)
 		(dnp no)
-		(property "Reference" "#PWR408"
+		(property "Reference" "#PWR0408"
 			(at 158.75 128.27 0)
 			(hide yes)
@@
 			(project "drum"
 				(path "/6c8448b4-b04d-47e1-934e-e40cbe27a7be/ba748654-beb9-4861-aa35-c19e08caaf2e"
-					(reference "#PWR408")
+					(reference "#PWR0408")
 					(unit 1)
 				)
@@
 		(in_pos_files yes)
 		(dnp no)
-		(property "Reference" "#PWR402"
+		(property "Reference" "#PWR0402"
 			(at 107.95 143.51 0)
 			(hide yes)
@@
 			(project "drum"
 				(path "/6c8448b4-b04d-47e1-934e-e40cbe27a7be/ba748654-beb9-4861-aa35-c19e08caaf2e"
-					(reference "#PWR402")
+					(reference "#PWR0402")
 					(unit 1)
 				)
@@
 		(in_pos_files yes)
 		(dnp no)
-		(property "Reference" "#PWR405"
+		(property "Reference" "#PWR0405"
 			(at 139.7 127 0)
 			(hide yes)
@@
 			(project "drum"
 				(path "/6c8448b4-b04d-47e1-934e-e40cbe27a7be/ba748654-beb9-4861-aa35-c19e08caaf2e"
-					(reference "#PWR405")
+					(reference "#PWR0405")
 					(unit 1)
 				)
