File: PWMChannel.kicad_sch (KiCad schematic)
At the start: 6 parts, among them J501 WAGO 2065-100, J502 WAGO 2065-100, Q501 BSC010N04LS

Commit message: Good Bye Imperial
Parts:
- C501: footprint V2_Capacitor_SMD:C_0603 -> V2_Capacitor_SMD:C_1608; symbol V2_Capacitor:0603_0u1 -> V2_Capacitor:1608_0u1
- Q501: Polarity (none) -> N
Changed lines of the file:
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@@
 	(title_block
 		(title "V2 drum")
-		(date "2026-04-14")
+		(date "2026-05-11")
 		(rev "2026-03-30")
 		(company "Versio Duo")
@@
 	)
 	(symbol
-		(lib_id "V2_Capacitor:0603_0u1")
+		(lib_id "V2_Capacitor:1608_0u1")
 		(at 116.84 86.36 0)
 		(unit 1)
@@
 			)
 		)
-		(property "Footprint" "V2_Capacitor_SMD:C_0603"
+		(property "Footprint" "V2_Capacitor_SMD:C_1608"
 			(at 116.84 103.378 0)
 			(hide yes)
@@
 			(hide yes)
 			(show_name no)
+			(do_not_autoplace no)
+			(effects
+				(font
+					(size 1.27 1.27)
+				)
+			)
+		)
+		(property "Polarity" "N"
+			(at 114.3 111.76 0)
+			(hide yes)
+			(show_name no)
