File: PowerSupply.kicad_sch (KiCad schematic)
At the start: 6 parts, among them U301 TPSM33620S5QRDNRQ1

Commit message: Good Bye Imperial
Parts:
- C301: footprint V2_Capacitor_SMD:C_1210 -> V2_Capacitor_SMD:C_3225; symbol V2_Capacitor:1210_10u -> V2_Capacitor:3225_10u
- C302: footprint V2_Capacitor_SMD:C_0603 -> V2_Capacitor_SMD:C_1608; symbol V2_Capacitor:0603_0u1 -> V2_Capacitor:1608_0u1
- C303: footprint V2_Capacitor_SMD:C_0603 -> V2_Capacitor_SMD:C_1608; symbol V2_Capacitor:0603_1u -> V2_Capacitor:1608_1u
- C304, C305: footprint V2_Capacitor_SMD:C_1210 -> V2_Capacitor_SMD:C_3225; symbol V2_Capacitor:1210_22u -> V2_Capacitor:3225_22u
Changed lines of the file:
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@@
 	(title_block
 		(title "V2 drum")
-		(date "2026-04-14")
+		(date "2026-05-11")
 		(rev "2026-03-30")
 		(company "Versio Duo")
@@
 	)
 	(symbol
-		(lib_id "V2_Capacitor:0603_0u1")
+		(lib_id "V2_Capacitor:1608_0u1")
 		(at 109.22 97.79 0)
 		(unit 1)
@@
 			)
 		)
-		(property "Footprint" "V2_Capacitor_SMD:C_0603"
+		(property "Footprint" "V2_Capacitor_SMD:C_1608"
 			(at 109.22 114.808 0)
 			(hide yes)
@@
 	)
 	(symbol
-		(lib_id "V2_Capacitor:1210_22u")
+		(lib_id "V2_Capacitor:3225_22u")
 		(at 195.58 97.79 0)
 		(unit 1)
@@
 			)
 		)
-		(property "Footprint" "V2_Capacitor_SMD:C_1210"
+		(property "Footprint" "V2_Capacitor_SMD:C_3225"
 			(at 195.58 114.808 0)
 			(hide yes)
@@
 	)
 	(symbol
-		(lib_id "V2_Capacitor:0603_1u")
+		(lib_id "V2_Capacitor:1608_1u")
 		(at 125.73 105.41 270)
 		(unit 1)
@@
 			)
 		)
-		(property "Footprint" "V2_Capacitor_SMD:C_0603"
+		(property "Footprint" "V2_Capacitor_SMD:C_1608"
 			(at 108.712 105.41 0)
 			(hide yes)
@@
 	)
 	(symbol
-		(lib_id "V2_Capacitor:1210_22u")
+		(lib_id "V2_Capacitor:3225_22u")
 		(at 185.42 97.79 0)
 		(unit 1)
@@
 			)
 		)
-		(property "Footprint" "V2_Capacitor_SMD:C_1210"
+		(property "Footprint" "V2_Capacitor_SMD:C_3225"
 			(at 185.42 114.808 0)
 			(hide yes)
@@
 	)
 	(symbol
-		(lib_id "V2_Capacitor:1210_10u")
+		(lib_id "V2_Capacitor:3225_10u")
 		(at 97.79 97.79 0)
 		(unit 1)
@@
 			)
 		)
-		(property "Footprint" "V2_Capacitor_SMD:C_1210"
+		(property "Footprint" "V2_Capacitor_SMD:C_3225"
 			(at 97.79 114.808 0)
 			(hide yes)
