File: drum.kicad_pcb (KiCad board)
At the start: 6 copper layers, 70 x 70 mm, 111 parts, among them J1001 NE8FAV, J101 Cortex, J102 DX07S016JA3, J501 WAGO 2065-100, J502 WAGO 2065-100, J601 WAGO 2065-100, J602 WAGO 2065-100, J701 WAGO 2065-100, J702 WAGO 2065-100, J703 WAGO 2065-100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

Commit message: Refresh
Parts:
- moved FID103 68.0 mm to (121.0, 71.0)
- moved INFO102 0.75 mm to (155.0, 137.8)
