File: drum.kicad_pcb (KiCad board)
At the start: 6 copper layers, 70 x 70 mm, 111 parts, among them J1001 NE8FAV, J101 Cortex, J102 DX07S016JA3, J501 WAGO 2065-100, J502 WAGO 2065-100, J601 WAGO 2065-100, J602 WAGO 2065-100, J701 WAGO 2065-100, J702 WAGO 2065-100, J703 WAGO 2065-100, J704 WAGO 2065-100, J801 WAGO 2065-100, J802 WAGO 2065-100, J803 WAGO 2065-100, J901 NE8FAV, Q201 BSC010N04LS, Q202 BSC010N04LS, Q501 BSC010N04LS, Q601 BSC010N04LS, SW101 SKSG, SW102 SKSG, U1001 THVD2442, U101 TPS78433QWDRBRQ1, U102 ATSAMD51J, U201 LM74502-Q1, U301 TPSM33620S5QRDNRQ1, U401 BTT6010, U701 TMC2130-LA, U801 74AHC1G125, U901 THVD2442, Y101 32k768

Commit message: Refresh
Connections:
- net /LED-PWM1 renamed /LED-PWM
- net /PWM-Power renamed /+VPWM
- net /PWM1 renamed /PWM-1
- net /PWM2 renamed /PWM-2
- U101 pad 6: unconnected-(U101-Pad6) -> +5V

Commit message: Rename
Connections:
- net /LED Strip/WS2812-data renamed /LED/WS2812-data
