File: Polarity-Protection.kicad_sch (KiCad schematic)
At the start: 6 parts, among them J501 WAGO 2065-100, J502 WAGO 2065-100, Q501 BSC010N04LS

Commit message: Rename
Parts:
- removed C501: 0u1, V2_Capacitor_SMD:C_1608, symbol V2_Capacitor:1608_0u1
- removed D501: PMEG6030AEXEX, V2_Diode_SMD:D_SOD-123HP, symbol V2_Diode:PMEG6030AEXEX
- removed D502: WS2812, V2_LED:WS2812-2020, symbol V2_LED:WS2812
- removed J501, J502: WAGO 2065-100, V2_Connector_WAGO:2065-100, symbol V2_Connector_WAGO:2065
- removed Q501: BSC010N04LS, V2_Package_TO_SOT_SMD:TDSON-8-FL, symbol V2_Transistor_FET:BSC010N04LS
- added C201: 0u1, V2_Capacitor_SMD:C_1608, symbol V2_Capacitor:1608_0u1
- added C202: 0u22, V2_Capacitor_SMD:C_1608, symbol V2_Capacitor:1608_0u22
- added Q201, Q202: BSC010N04LS, V2_Package_TO_SOT_SMD:TDSON-8-FL, symbol V2_Transistor_FET:BSC010N04LS
- added R201: 100k, V2_Resistor_SMD:R_1608, symbol V2_Resistor:1608_100k
- added R202: 3k9, V2_Resistor_SMD:R_1608, symbol V2_Resistor:1608_3k9
- added U201: LM74502-Q1, V2_Package_TO_SOT_SMD:SOT-23-8, symbol V2_Power_Management:LM74502-Q1
Connections:
- net GND: now also C201.2, R202.2, U201.2 (GND)
- new net: C202.2, U201.4 (VCAP)
- new net Gate: Q201.4 (G), Q202.4 (G), U201.6 (GATE)
- new net Input: C201.1, C202.1, Q201.5 (D), R201.1, U201.1 (EN/UVLO), U201.5 (VS)
- new net Output: Q202.5 (D)
- new net Overvoltage: R201.2, R202.1, U201.7 (OV)
- new net Source: Q201.1 (S), Q202.1 (S), U201.8 (SRC)
Other:
- note added: "(100kΩ + 3.9kΩ) × 1.25V (threshold) ------------------------ = 33.3V Overvoltage Protection 3.9kΩ"
