File: Power-DCDC.kicad_sch (KiCad schematic)
At the start: 7 parts, among them Q201 BSC010N04LS, Q202 BSC010N04LS, U201 LM74502-Q1

Commit message: Rename
Parts:
- removed C201: 0u1, V2_Capacitor_SMD:C_1608, symbol V2_Capacitor:1608_0u1
- removed C202: 0u22, V2_Capacitor_SMD:C_1608, symbol V2_Capacitor:1608_0u22
- removed Q201, Q202: BSC010N04LS, V2_Package_TO_SOT_SMD:TDSON-8-FL, symbol V2_Transistor_FET:BSC010N04LS
- removed R201: 100k, V2_Resistor_SMD:R_1608, symbol V2_Resistor:1608_100k
- removed R202: 3k9, V2_Resistor_SMD:R_1608, symbol V2_Resistor:1608_3k9
- removed U201: LM74502-Q1, V2_Package_TO_SOT_SMD:SOT-23-8, symbol V2_Power_Management:LM74502-Q1
- added C301: 10u, V2_Capacitor_SMD:C_3225, symbol V2_Capacitor:3225_10u
- added C302: 0u1, V2_Capacitor_SMD:C_1608, symbol V2_Capacitor:1608_0u1
- added C303: 1u, V2_Capacitor_SMD:C_1608, symbol V2_Capacitor:1608_1u
- added C304, C305: 22u, V2_Capacitor_SMD:C_3225, symbol V2_Capacitor:3225_22u
- added U301: TPSM33620S5QRDNRQ1, V2_Converter_DCDC:QFN-11, symbol V2_Converter_DCDC:TPSM33620S5QRDNRQ1
Connections:
- net GND: now also C301.2, C302.2, C303.2, C304.2, C305.2, U301.10 (GND), U301.11 (MODE)
- net Input: now also C301.1, C302.1, U301.2 (EN), U301.3 (VIN)
- new net +5V: C304.1, C305.1, U301.4 (VOUT), U301.9 (FB)
- new net Vcc: C303.1, U301.8 (VCC)
- no-connect marks 0 -> 1
Other:
- note removed: "(100kΩ + 3.9kΩ) × 1.25V (threshold) ------------------------ = 33.3V Overvoltage Protection 3.9kΩ"
