File: drum.kicad_sch (KiCad schematic)
At the start: 39 parts, among them J101 Cortex, J102 DX07S016JA3, SW101 SKSG, SW102 SKSG, U101 TPS78433QWDRBRQ1, U102 ATSAMD51J, Y101 32k768

Commit message: Refresh
Connections:
- net +5V: now also U101.6 (EN)
- net LED-PWM1 renamed LED-PWM
- net PWM1 renamed PWM-1
- net PWM2 renamed PWM-2
Other:
- sheet PWM Power ports: added +VPWM; removed Power

Commit message: Rename
Other:
- sheet LED Strip renamed LED
- sheet LED: file LEDStrip.kicad_sch -> LED.kicad_sch
- sheet Link Plug: file LinkPlug.kicad_sch -> Link-Plug.kicad_sch
- sheet Link Socket: file LinkSocket.kicad_sch -> Link-Socket.kicad_sch
- sheet PWM Channel 1: file PWMChannel.kicad_sch -> PWM-Channel.kicad_sch
- sheet PWM Channel 2: file PWMChannel.kicad_sch -> PWM-Channel.kicad_sch
- sheet PWM Power: file PowerSwitch.kicad_sch -> Power-Switch.kicad_sch
- sheet Polarity Protection: file PolarityProtection.kicad_sch -> Polarity-Protection.kicad_sch
- sheet Power +5V: file PowerSupply.kicad_sch -> Power-DCDC.kicad_sch
- sheet Stepper: file StepperDriver.kicad_sch -> Stepper.kicad_sch
Changed lines of the file:
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@@
 	(title_block
 		(title "V2 drum")
-		(date "2026-08-28")
+		(date "2026-08-30")
 		(rev "2026-05-25")
 		(company "Versio Duo")
@@
 		(unit 1)
 		(body_style 1)
-		(exclude_from_sim no)
+		(exclude_from_sim yes)
 		(in_bom no)
 		(on_board yes)
@@
 			)
 		)
-		(property "Sim.Enable" "0"
-			(at 240.03 170.18 0)
-			(hide yes)
-			(show_name no)
-			(do_not_autoplace no)
-			(effects
-				(font
-					(size 1.27 1.27)
-				)
-			)
-		)
 		(instances
 			(project "drum"
@@
 		(unit 1)
 		(body_style 1)
-		(exclude_from_sim no)
+		(exclude_from_sim yes)
 		(in_bom no)
 		(on_board yes)
@@
 			)
 		)
-		(property "Sim.Enable" "0"
-			(at 227.33 180.34 0)
-			(hide yes)
-			(show_name no)
-			(do_not_autoplace no)
-			(effects
-				(font
-					(size 1.27 1.27)
-				)
-			)
-		)
 		(instances
 			(project "drum"
@@
 		(unit 1)
 		(body_style 1)
-		(exclude_from_sim no)
+		(exclude_from_sim yes)
 		(in_bom no)
 		(on_board yes)
@@
 			)
 		)
-		(property "Sim.Enable" "0"
-			(at 240.03 165.1 0)
-			(hide yes)
-			(show_name no)
-			(do_not_autoplace no)
-			(effects
-				(font
-					(size 1.27 1.27)
-				)
-			)
-		)
 		(instances
 			(project "drum"
@@
 			)
 		)
-		(property "Sheetfile" "LinkSocket.kicad_sch"
+		(property "Sheetfile" "Link-Socket.kicad_sch"
 			(at 266.7 155.5246 0)
 			(hide yes)
@@
 			)
 		)
-		(property "Sheetfile" "StepperDriver.kicad_sch"
+		(property "Sheetfile" "Stepper.kicad_sch"
 			(at 193.04 93.2946 0)
 			(hide yes)
@@
 			(color 255 255 194 1)
 		)
-		(property "Sheetname" "LED Strip"
+		(property "Sheetname" "LED"
 			(at 261.62 78.0284 0)
 			(show_name no)
@@
 			)
 		)
-		(property "Sheetfile" "LEDStrip.kicad_sch"
+		(property "Sheetfile" "LED.kicad_sch"
 			(at 261.62 84.4046 0)
 			(hide yes)
@@
 			)
 		)
-		(property "Sheetfile" "PowerSwitch.kicad_sch"
+		(property "Sheetfile" "Power-Switch.kicad_sch"
 			(at 223.52 37.4146 0)
 			(hide yes)
@@
 			)
 		)
-		(property "Sheetfile" "PWMChannel.kicad_sch"
+		(property "Sheetfile" "PWM-Channel.kicad_sch"
 			(at 248.92 53.9246 0)
 			(hide yes)
@@
 			)
 		)
-		(property "Sheetfile" "LinkPlug.kicad_sch"
+		(property "Sheetfile" "Link-Plug.kicad_sch"
 			(at 266.7 119.9646 0)
 			(hide yes)
@@
 			)
 		)
-		(property "Sheetfile" "PolarityProtection.kicad_sch"
+		(property "Sheetfile" "Polarity-Protection.kicad_sch"
 			(at 172.72 46.3046 0)
 			(hide yes)
@@
 			)
 		)
-		(property "Sheetfile" "PowerSupply.kicad_sch"
+		(property "Sheetfile" "Power-DCDC.kicad_sch"
 			(at 34.29 156.7946 0)
 			(hide yes)
@@
 			)
 		)
-		(property "Sheetfile" "PWMChannel.kicad_sch"
+		(property "Sheetfile" "PWM-Channel.kicad_sch"
 			(at 214.63 53.9246 0)
 			(hide yes)
